File: PCB/Rear_Light_v1.kicad_pcb (KiCad board)
At the start: 2 copper layers, 32 x 20.3 mm, 29 parts, among them J1 USB_B_Micro, Q1 si2302, SW1 SW_Push, U1 TP4056, U2 N76E003AQ20, U3 SC662K

Commit message: chematic + pcb added
Parts:
- moved BAT+1 55.6 mm to (113.1, 102.0)
- moved BAT-1 55.6 mm to (113.1, 98.5)
- moved Q1 55.6 mm to (103.8, 110.2)
- moved R1 55.6 mm to (109.6, 98.0)
- moved R4 55.6 mm to (103.8, 112.7)
- moved R5 55.6 mm to (103.8, 114.2)
- moved RN1 55.6 mm to (88.1, 108.3)
- moved SW1 55.6 mm to (108.7, 106.4)
- moved TH1 55.6 mm to (98.8, 98.0)
- moved AC1 55.6 mm to (92.5, 108.7)
- moved C1 55.6 mm to (98.8, 102.2)
- moved C2 55.6 mm to (109.6, 102.2)
- moved C3 55.6 mm to (90.3, 114.8)
- moved C4 55.6 mm to (95.1, 101.7)
- moved D1 55.6 mm to (109.6, 100.8)
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Connections:
- U2 pad 7: (no net) -> /LED_gate
- U2 pad 8: /LED_gate -> /light(analog)
- U2 pad 9: /light(analog) -> (no net)
Other:
- board text added: "to do: move light to ADC pin"
